File: ClickerController/_autosave-ClickerController.kicad_pcb (KiCad board)
At the start: 2 copper layers, 42.7 x 40.9 mm, 12 parts, among them J1 Screw_Terminal_01x02, J2 Screw_Terminal_01x03, J3 Conn_01x10_Male, J4 Conn_01x04_Male, U1 CD74HC4067M, U2 CD74HC4067M, U3 74HC595

Commit message: Add files via upload
Parts:
- added REF**: MountingHole_3.2mm_M3, MountingHole:MountingHole_3.2mm_M3, F.Cu at (162.3, 94.0)
- moved REF** 31.7 mm to (136.9, 94.0)
- moved J1 9.57 mm to (134.4, 82.6)
- moved J2 5.62 mm to (153.4, 96.5), turned to -90 degrees
Routing:
- net SRCLK: track 22.0 -> 5.93 mm
- net RCLK: track 16.4 -> 7.58 mm
- net 5v: track 88.8 -> 92.3 mm
- net SER: track 10.8 -> 12.2 mm
Other:
- board size 42.7 x 40.9 mm -> 42.7 x 42.7 mm
Changed lines of the file:
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@@
   (net 49 "unconnected-(U2-Pad23)")
   (footprint "Connector_PinHeader_2.54mm:PinHeader_1x03_P2.54mm_Vertical" (layer "F.Cu")
-    (at 156.845 92.075 90)
+    (at 153.401 96.52 -90)
     (descr "Through hole straight pin header, 1x03, 2.54mm pitch, single row")
     (tags "Through hole pin header THT 1x03 2.54mm single row")
@@
     (fp_line (start -0.635 -1.27) (end 1.27 -1.27) (layer "F.Fab") (width 0.1))
     (fp_line (start -1.27 6.35) (end -1.27 -0.635) (layer "F.Fab") (width 0.1))
-    (pad "1" thru_hole rect (at 0 0 90) (size 1.7 1.7) (drill 1) (layers *.Cu *.Mask)
+    (pad "1" thru_hole rect (at 0 0 270) (size 1.7 1.7) (drill 1) (layers *.Cu *.Mask)
       (net 3 "SER") (pinfunction "Pin_1") (pintype "passive"))
-    (pad "2" thru_hole oval (at 0 2.54 90) (size 1.7 1.7) (drill 1) (layers *.Cu *.Mask)
+    (pad "2" thru_hole oval (at 0 2.54 270) (size 1.7 1.7) (drill 1) (layers *.Cu *.Mask)
       (net 5 "RCLK") (pinfunction "Pin_2") (pintype "passive"))
-    (pad "3" thru_hole oval (at 0 5.08 90) (size 1.7 1.7) (drill 1) (layers *.Cu *.Mask)
+    (pad "3" thru_hole oval (at 0 5.08 270) (size 1.7 1.7) (drill 1) (layers *.Cu *.Mask)
       (net 4 "SRCLK") (pinfunction "Pin_3") (pintype "passive"))
     (model "${KICAD6_3DMODEL_DIR}/Connector_PinHeader_2.54mm.3dshapes/PinHeader_1x03_P2.54mm_Vertical.wrl"
@@
   )
   (footprint "MountingHole:MountingHole_3.2mm_M3" (layer "F.Cu")
-    (at 107.696 81.788)
+    (at 136.906 93.98)
     (descr "Mounting Hole 3.2mm, no annular, M3")
     (tags "mounting hole 3.2mm no annular m3")
@@
     )
   )
+  (footprint "MountingHole:MountingHole_3.2mm_M3" (layer "F.Cu")
+    (at 162.306 93.98)
+    (descr "Mounting Hole 3.2mm, no annular, M3")
+    (tags "mounting hole 3.2mm no annular m3")
+    (attr exclude_from_pos_files exclude_from_bom)
+    (fp_text reference "REF**" (at 0 -4.2) (layer "F.SilkS")
+      (effects (font (size 1 1) (thickness 0.15)))
+    )
+    (fp_text value "MountingHole_3.2mm_M3" (at 0 4.2) (layer "F.Fab")
+      (effects (font (size 1 1) (thickness 0.15)))
+    )
+    (fp_text user "${REFERENCE}" (at 0 0) (layer "F.Fab")
+      (effects (font (size 1 1) (thickness 0.15)))
+    )
+    (fp_circle (center 0 0) (end 3.2 0) (layer "Cmts.User") (width 0.15) (fill none))
+    (fp_circle (center 0 0) (end 3.45 0) (layer "F.CrtYd") (width 0.05) (fill none))
+    (pad "" np_thru_hole circle (at 0 0) (size 3.2 3.2) (drill 3.2) (layers F&B.Cu *.Mask))
+  )
   (footprint "Connector_PinHeader_2.54mm:PinHeader_1x02_P2.54mm_Vertical" (layer "F.Cu")
-    (at 135.255 92.08 180)
+    (at 134.366 82.555 180)
     (descr "Through hole straight pin header, 1x02, 2.54mm pitch, single row")
     (tags "Through hole pin header THT 1x02 2.54mm single row")
@@
     )
   )
-  (gr_rect (start 131.064 57.404) (end 173.736 98.298) (layer "Edge.Cuts") (width 0.1) (fill none))
+  (gr_rect (start 131.064 57.404) (end 173.736 100.076) (layer "Edge.Cuts") (width 0.1) (fill none))
   (gr_text "Controller V1\n2023 - Freaughouse" (at 159.385 64.77) (layer "B.SilkS")
     (effects (font (size 1 1) (thickness 0.15)) (justify mirror))
@@
   (via (at 140.97 82.55) (size 0.8) (drill 0.4) (layers "F.Cu" "B.Cu") (net 1))
   (via (at 142.24 87.63) (size 0.8) (drill 0.4) (layers "F.Cu" "B.Cu") (net 1))
-  (segment (start 135.255 92.71) (end 135.255 92.08) (width 0.25) (layer "F.Cu") (net 2))
+  (segment (start 140.716 88.9) (end 140.716 87.376) (width 0.25) (layer "F.Cu") (net 2))
+  (segment (start 141.224 89.408) (end 140.716 88.9) (width 0.25) (layer "F.Cu") (net 2))
   (segment (start 152.974 68.58) (end 153.228 68.326) (width 0.25) (layer "F.Cu") (net 2))
-  (segment (start 143.51 92.71) (end 143.51 95.25) (width 0.25) (layer "F.Cu") (net 2))
-  (segment (start 138.43 95.885) (end 135.255 92.71) (width 0.25) (layer "F.Cu") (net 2))
-  (segment (start 143.51 95.25) (end 142.875 95.885) (width 0.25) (layer "F.Cu") (net 2))
+  (segment (start 138.684 86.868) (end 137.16 85.344) (width 0.25) (layer "F.Cu") (net 2))
+  (segment (start 143.51 90.424) (end 142.494 89.408) (width 0.25) (layer "F.Cu") (net 2))
   (segment (start 170.815 86.675) (end 170.815 84.66) (width 0.25) (layer "F.Cu") (net 2))
-  (segment (start 142.875 95.885) (end 138.43 95.885) (width 0.25) (layer "F.Cu") (net 2))
+  (segment (start 136.149 82.555) (end 134.366 82.555) (width 0.25) (layer "F.Cu") (net 2))
+  (segment (start 137.16 83.566) (end 136.149 82.555) (width 0.25) (layer "F.Cu") (net 2))
+  (segment (start 140.716 87.376) (end 140.208 86.868) (width 0.25) (layer "F.Cu") (net 2))
+  (segment (start 142.494 89.408) (end 141.224 89.408) (width 0.25) (layer "F.Cu") (net 2))
+  (segment (start 143.51 92.645) (end 143.51 90.424) (width 0.25) (layer "F.Cu") (net 2))
+  (segment (start 140.208 86.868) (end 138.684 86.868) (width 0.25) (layer "F.Cu") (net 2))
   (segment (start 150.7 68.58) (end 152.974 68.58) (width 0.25) (layer "F.Cu") (net 2))
   (segment (start 143.51 92.645) (end 143.51 92.71) (width 0.25) (layer "F.Cu") (net 2))
+  (segment (start 137.16 85.344) (end 137.16 83.566) (width 0.25) (layer "F.Cu") (net 2))
   (via (at 170.815 84.455) (size 0.8) (drill 0.4) (layers "F.Cu" "B.Cu") (net 2))
   (via (at 151.13 92.71) (size 0.8) (drill 0.4) (layers "F.Cu" "B.Cu") (net 2))
@@
   (segment (start 149.975 67.855) (end 141.304695 67.855) (width 0.25) (layer "B.Cu") (net 2))
   (segment (start 150.7 68.58) (end 149.975 67.855) (width 0.25) (layer "B.Cu") (net 2))
-  (segment (start 155.575 92.075) (end 153.67 90.17) (width 0.25) (layer "F.Cu") (net 3))
+  (segment (start 148.59 91.44) (end 148.59 92.645) (width 0.25) (layer "F.Cu") (net 3))
   (segment (start 149.86 90.17) (end 148.59 91.44) (width 0.25) (layer "F.Cu") (net 3))
-  (segment (start 153.67 90.17) (end 149.86 90.17) (width 0.25) (layer "F.Cu") (net 3))
-  (segment (start 148.59 91.44) (end 148.59 92.645) (width 0.25) (layer "F.Cu") (net 3))
-  (segment (start 156.845 92.075) (end 155.575 92.075) (width 0.25) (layer "F.Cu") (net 3))
-  (segment (start 160.02 95.885) (end 146.685 95.885) (width 0.25) (layer "F.Cu") (net 4))
-  (segment (start 146.685 95.885) (end 144.78 93.98) (width 0.25) (layer "F.Cu") (net 4))
+  (segment (start 152.146 90.17) (end 149.86 90.17) (width 0.25) (layer "F.Cu") (net 3))
+  (segment (start 153.401 96.52) (end 153.401 91.425) (width 0.25) (layer "F.Cu") (net 3))
+  (segment (start 153.401 91.425) (end 152.146 90.17) (width 0.25) (layer "F.Cu") (net 3))
+  (segment (start 147.32 96.52) (end 144.78 93.98) (width 0.25) (layer "F.Cu") (net 4))
   (segment (start 144.78 93.98) (end 144.78 92.645) (width 0.25) (layer "F.Cu") (net 4))
-  (segment (start 161.925 92.075) (end 161.925 93.98) (width 0.25) (layer "F.Cu") (net 4))
-  (segment (start 161.925 93.98) (end 160.02 95.885) (width 0.25) (layer "F.Cu") (net 4))
-  (segment (start 158.115 94.615) (end 147.32 94.615) (width 0.25) (layer "F.Cu") (net 5))
+  (segment (start 148.321 96.52) (end 147.32 96.52) (width 0.25) (layer "F.Cu") (net 4))
   (segment (start 147.32 94.615) (end 146.05 93.345) (width 0.25) (layer "F.Cu") (net 5))
-  (segment (start 159.385 93.345) (end 158.115 94.615) (width 0.25) (layer "F.Cu") (net 5))
-  (segment (start 159.385 92.075) (end 159.385 93.345) (width 0.25) (layer "F.Cu") (net 5))
+  (segment (start 150.861 95.235) (end 150.241 94.615) (width 0.25) (layer "F.Cu") (net 5))
+  (segment (start 150.241 94.615) (end 147.32 94.615) (width 0.25) (layer "F.Cu") (net 5))
+  (segment (start 150.861 96.52) (end 150.861 95.235) (width 0.25) (layer "F.Cu") (net 5))
   (segment (start 146.05 93.345) (end 146.05 92.645) (width 0.25) (layer "F.Cu") (net 5))
   (segment (start 160.02 70.485) (end 160.02 60.96) (width 0.25) (layer "F.Cu") (net 6))
@@
     (polygon
       (pts
-        (xy 173.355 97.79)
-        (xy 131.445 97.79)
+        (xy 173.355 99.568)
+        (xy 131.445 99.568)
         (xy 131.445 57.785)
         (xy 173.355 57.785)
@@
     (polygon
       (pts
-        (xy 172.085 95.885)
-        (xy 132.715 95.885)
+        (xy 172.085 98.425)
+        (xy 132.715 98.425)
         (xy 132.715 59.69)
         (xy 172.085 59.69)
